File: RSC_extension_board.kicad_sch (KiCad schematic)
At the start: 39 parts, among them J1 Conn_01x03, J10 Conn_01x02, J13 Conn_01x03, J14 500SSP1S2M2QEA, J16 Conn_01x07, J2 Conn_01x03, J3 Raspberry_Pi_4, J4 Conn_01x04, J5 Conn_01x03, J6 Conn_01x02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

Commit message: spi display pinout change. button connector simplified.
Parts:
- removed D1, D2: PJSD03TS-AU_R1_000A1, SODFL1608X65N, symbol PJSD03TS-AU_R1_000A1:PJSD03TS-AU_R1_000A1
- removed J16: Conn_01x07, Connector_PinSocket_2.54mm:PinSocket_1x07_P2.54mm_Vertical, symbol Connector_Generic:Conn_01x07
- removed R3, R4: 10k, Resistor_SMD:R_0603_1608Metric_Pad0.98x0.95mm_HandSolder, symbol Device:R
- added C37: 100nF, Capacitor_SMD:C_0603_1608Metric_Pad1.08x0.95mm_HandSolder, symbol Device:C
- added J16: Conn_01x10, Connector_PinSocket_2.54mm:PinSocket_1x10_P2.54mm_Vertical, symbol Connector_Generic:Conn_01x10
Connections:
- net +3.3V: now also J16.1 (Pin_1)
- net +5V: now also C37.1, J16.10 (Pin_10)
- net BUTTON: now also J6.1 (Pin_1)
- net Earth: now also C37.2, J16.2 (Pin_2)
- net SPI_DC: now reaches J3.13 (GPIO27/SDIO_DAT3)
- net SPI_DC: now also J16.8 (Pin_8)
- net LCD_BL: now reaches J3.15 (GPIO22/SDIO_CLK)
- net LCD_BL: now also J16.7 (Pin_7)
- net SPI_RST: now reaches J3.7 (GPCLK0/GPIO04)
- net SPI_RST: now also J16.3 (Pin_3)
- net at D3.3, F1.1, J9.A9 (VBUS)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: no longer U1.5 (VBUS)
- net GPIO07: no longer names the net of J3.26 (~{CE1}_SPI0/GPIO07)
- net GPIO08 renamed SPI_CS
- net SPI_CS: now also J16.4 (Pin_4)
- net GPIO09 renamed SPI_MISO
- net SPI_MISO: now also J16.9 (Pin_9)
- net GPIO10 renamed SPI_MOSI
- net SPI_MOSI: now also J16.5 (Pin_5)
- net GPIO11 renamed SPI_CLK
- net SPI_CLK: now also J16.6 (Pin_6)
- no-connect marks 0 -> 1
Other:
- note added: "Intended for Adafruit Mini LED Arcade Button - 24mm Translucent Clear with built in current limiting. https://www.adafruit.com/product/3429"
- note added: "Needs to be modified for 5V"
- moved on the sheet: C36, C5, J6, J8
