File: voice.kicad_sch (KiCad schematic)
At the start: 43 parts, among them J14 Conn_01x02, J15 Conn_01x02, SW1 SW_Wuerth_450301014042, U1 WM8960CGEFL_V, U2 AP2112K-3.3, Y1 ECS-3225MV

Commit message: update sch
Other:
- title: RSC hat board -> RSC hat board - TorxHAT
Changed lines of the file:
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@@
 	(paper "A4")
 	(title_block
-		(title "RSC hat board")
-		(date "2026-06-01")
-		(rev "A")
-		(comment 1 "Author: Raiko Torga")
+		(title "RSC hat board - TorxHAT")
+		(date "2026-07-17")
+		(rev "B")
+		(comment 1 "Authors: Raiko Torga, Matevz B. Zorec")
 	)
 	(text "This circuit is based on the Adafruit Voice Bonnet schematic design:\nhttps://github.com/adafruit/Adafruit-Voice-Bonnet-PCB/blob/master/Adafruit%20Voice%20Bonnet.sch\n"

Commit message: progress alhamdulliah... last batch = buck stage patches + thermal via spam
Connections:
- no-connect marks 0 -> 7
Changed lines of the file:
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@@
 		(color 0 0 0 0)
+	)
+	(no_connect
+		(at 107.95 162.56)
+	)
+	(no_connect
+		(at 107.95 160.02)
+	)
+	(no_connect
+		(at 107.95 152.4)
+	)
+	(no_connect
+		(at 107.95 144.78)
+	)
+	(no_connect
+		(at 107.95 157.48)
+	)
+	(no_connect
+		(at 107.95 142.24)
+	)
+	(no_connect
+		(at 107.95 154.94)
 	)
 	(wire
