File: USB_power.kicad_sch (KiCad schematic)
At the start: 30 parts, among them J16 USB_C_Receptacle_PowerOnly_6P, Q3 DMP3013SFV, Q4 DMP3013SFV, U5 CYPD3177-24LQ

Commit message: WIP - need to validate revA neopx working at curr pin
Parts:
- R10: value DNP -> 1k; now fitted
- R12, R9: value 0 -> 5.1k
- R13: value DNP -> 5.1k; now fitted

Commit message: update sch
Parts:
- R10: value 1k -> DNP; now not fitted
- R12, R9: value 5.1k -> 0
- R13: value 5.1k -> DNP; now not fitted
- R17: value 1k -> 68
Other:
- title: RSC hat board -> RSC hat board - TorxHAT
Changed lines of the file:
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@@
 	(paper "A4")
 	(title_block
-		(title "RSC hat board")
-		(date "2026-06-01")
-		(rev "A")
-		(comment 1 "Author: Raiko Torga")
+		(title "RSC hat board - TorxHAT")
+		(date "2026-07-17")
+		(rev "B")
+		(comment 1 "Authors: Raiko Torga, Matevz B. Zorec")
 	)
 	(text "20V 2.5A\nhttps://www.infineon.com/assets/row/public/documents/24/49/\ninfineon-ez-pd-bcr-datasheet-usb-type-c-port-controller-for-power-sinks-datasheet-en.pdf"
@@
 			)
 		)
-		(property "Value" "1k"
+		(property "Value" "68"
 			(at 160.02 99.06 90)
 			(show_name no)
@@
 		(on_board yes)
 		(in_pos_files yes)
-		(dnp no)
+		(dnp yes)
 		(fields_autoplaced yes)
 		(property "Reference" "R13"
@@
 			)
 		)
-		(property "Value" "5.1k"
+		(property "Value" "DNP"
 			(at 129.54 153.6699 0)
 			(show_name no)
@@
 			)
 		)
-		(property "Value" "5.1k"
+		(property "Value" "0"
 			(at 129.54 143.5099 0)
 			(show_name no)
@@
 		(on_board yes)
 		(in_pos_files yes)
-		(dnp no)
+		(dnp yes)
 		(fields_autoplaced yes)
 		(property "Reference" "R10"
@@
 			)
 		)
-		(property "Value" "1k"
+		(property "Value" "DNP"
 			(at 111.76 153.6699 0)
 			(show_name no)
@@
 			)
 		)
-		(property "Value" "5.1k"
+		(property "Value" "0"
 			(at 111.76 143.5099 0)
 			(show_name no)

Commit message: update
Parts:
- R10: value DNP -> 1k; now fitted
- R12, R9: value 0 -> 5.1k
- R13: value DNP -> 5.1k; now fitted
Changed lines of the file:
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@@
 		(on_board yes)
 		(in_pos_files yes)
-		(dnp yes)
+		(dnp no)
 		(fields_autoplaced yes)
 		(property "Reference" "R13"
@@
 			)
 		)
-		(property "Value" "DNP"
+		(property "Value" "5.1k"
 			(at 129.54 153.6699 0)
 			(show_name no)
@@
 			)
 		)
-		(property "Value" "0"
+		(property "Value" "5.1k"
 			(at 129.54 143.5099 0)
 			(show_name no)
@@
 		(on_board yes)
 		(in_pos_files yes)
-		(dnp yes)
+		(dnp no)
 		(fields_autoplaced yes)
 		(property "Reference" "R10"
@@
 			)
 		)
-		(property "Value" "DNP"
+		(property "Value" "1k"
 			(at 111.76 153.6699 0)
 			(show_name no)
@@
 			)
 		)
-		(property "Value" "0"
+		(property "Value" "5.1k"
 			(at 111.76 143.5099 0)
 			(show_name no)

Commit message: update; add EN servo rail ctrl via GPIO05
Parts:
- added C56: 100uF, Capacitor_SMD:C_0603_1608Metric_Pad1.08x0.95mm_HandSolder, symbol Device:C
Connections:
- net GND: now also C56.1
- net VBUS: now also C56.2
Other:
- note added: "Bulk Cap 25V"
- note added: "Config: 15V max & 9V min R9: 5.1kΩ (VBUS_MIN pull-up) R10: 1kΩ (VBUS_MIN pull-down) R12: 5.1kΩ (VBUS_MAX pull-up) R13: 5.1kΩ (VBUS_MAX pull-down)"
- moved on the sheet: C55
